File: grafix.kicad_pcb (KiCad board)
At the start: 2 copper layers, 30.5 x 38.1 mm, 9 parts, among them J1 U64, J2 U65, J3 CKPIX, U1 74LS153, U2 74LS153, U3 74LS175

Commit message: Minor tweaks
Routing:
- net Net-(J3-Pin_1): track 10.3 -> 9.04 mm
Changed lines of the file:
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@@
 	)
 	(segment
-		(start 124.841 33.02)
-		(end 127 33.02)
+		(start 124.841 35.941)
+		(end 128.27 39.37)
 		(width 0.508)
 		(layer "F.Cu")
@@
 	)
 	(segment
-		(start 127 33.02)
-		(end 128.27 34.29)
+		(start 124.841 33.02)
+		(end 124.841 35.941)
 		(width 0.508)
 		(layer "F.Cu")
@@
 	)
 	(segment
-		(start 128.27 34.29)
+		(start 128.27 39.37)
 		(end 128.27 40.64)
 		(width 0.508)
