File: grafix.kicad_sch (KiCad schematic)
At the start: 9 parts, among them J1 U64, J2 U65, J3 CKPIX, U1 74LS153, U2 74LS153, U3 74LS175

Commit message: Minor schematic fix
Other:
- company: (none) -> Przemysław Węgrzyn <pwegrzyn@codepainters.com>
- title: (none) -> GraFIX - pixel glitch eliminator for Elwro 800 Junior
- moved on the sheet: C1, C2, C3
